File: Hardware/ESP-Wroom-32/Wroom32.kicad_pcb (KiCad board)
At the start: 2 copper layers, 71.3 x 61 mm, 35 parts, among them J1 USB_C_Receptacle_USB2.0, Q1 MMBT3904, Q2 MMBT3904, SW1 SW_Push, SW2 SW_DIP_x01, U1 CH340G, U2 AMS1117-3.3, U3 ESP32-WROOM-32, Y1 12M

Commit message: ...
Other:
- board text added: "Yup... Seems it'll work for the ESP32-S3-Wroom-1 also..."
Changed lines of the file:
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@@
       (rotate (xyz 0 0 -90))
     )
-    (model "../(KiCAD Customs)/3D/ESP32/ESP-32 .step"
+    (model "../(KiCAD Customs)/3D/ESP32/ESP-32 .step" hide
       (offset (xyz 0 3 0))
       (scale (xyz 1 1 1))
@@
     (effects (font (size 1 1) (thickness 0.15)))
   )
+  (gr_text "Yup...\nSeems it'll work for the\nESP32-S3-Wroom-1\nalso..." (at 150.033236 83.948286) (layer "F.SilkS")
+    (effects (font (size 0.5 0.5) (thickness 0.125)))
+  )
   (gr_text "(If you can read this...\nYou forgot to assemble\nyour programmer.)" (at 185.56 110.16) (layer "F.SilkS")
