File: Hardware/ESP-12/ESP12.kicad_sch (KiCad schematic)
At the start: 24 parts, among them J1 USB_C_Receptacle_USB2.0, J2 Conn_01x06_Male, J3 Conn_01x06_Male, Q1 MMBT3904, Q2 MMBT3904, SW1 SW_Push, SW2 SW_DIP_x01, U1 CH340G, U2 AMS1117-3.3, Y1 12M

Commit message: Starting extensive schematic tidy-up
Parts:
- removed J3: Conn_01x06_Male, Connector_PinHeader_2.54mm:PinHeader_1x06_P2.54mm_Vertical, symbol Connector:Conn_01x06_Male
- removed SW2: SW_DIP_x01, Tinker:SW_DIP_SPSTx01_Slide_6.7x4.1mm_W7.62mm_P2.54mm_LowProfile, symbol Switch:SW_DIP_x01
- added SW?: SW_DIP_x01, Tinker:SW_DIP_SPSTx01_Slide_6.7x4.1mm_W7.62mm_P2.54mm_LowProfile, symbol Switch:SW_DIP_x01
Connections:
- net +3.3V: now also SW?.2
- net Vsw: now also SW?.1
Other:
- note added: "Standalone"
- company: (none) -> ESP-12/07 Edition
- title: (none) -> The Nerd Mage Module Programmer
- moved on the sheet: C1, C2, C3, C4, C5, D1, D2, J2, Q1, Q2, R1, R2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
