File: Hardware/ESP-12/ESP12.kicad_sch (KiCad schematic)
At the start: 23 parts, among them J1 USB_C_Receptacle_USB2.0, J2 Conn_01x06_Male, Q1 MMBT3904, Q2 MMBT3904, SW1 SW_Push, U1 CH340G, U2 AMS1117-3.3, Y1 12M

Commit message: Getting up to rev 1
Parts:
- added R7, R8: 10K, Tinker:R_0603_1608Metric_Pad0.98x0.95mm_HandSolder, symbol Device:R
- gave numbers to parts that had none: 1
Connections:
- net +3.3V: now also D2.2 (A), R1.1, R2.1, Um1.8 (Vcc), R8.1; no longer SW2.2
- net GND: now also SW2.1; no longer R6.2, Um1.9 (GND)
- net Vsw: no longer D2.2 (A), R1.1, R2.1, SW2.1, Um1.8 (Vcc)
- net io0: now also R8.2
- net io15: now reaches Um1.10 ((MTDO)_GPIO15)
- net io15: now also R7.1
- new net mGND: R6.2, R7.2, SW2.2, Um1.9 (GND)
Other:
- moved on the sheet: R2, SW2

Commit message: updating sheet info
Other:
- note added: "Power"
- note removed: "V-REG"
- company: ESP-12/07 Edition -> S. A. Miller
- moved on the sheet: R2, R7
Changed lines of the file:
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@@
   (title_block
     (title "The Nerd Mage Module Programmer")
-    (rev "0.5.2")
-    (company "ESP-12/07 Edition")
+    (date "2023-07-13")
+    (rev "1.0.?")
+    (company "S. A. Miller")
+    (comment 1 "ESP-12/07 Edition")
   )
   (junction (at 83.82 64.77) (diameter 0) (color 0 0 0 0)
@@
     (stroke (width 0) (type default) (color 0 0 0 0))
   )
-  (wire (pts (xy 134.62 46.99) (xy 134.62 52.07))
-    (stroke (width 0) (type default) (color 0 0 0 0))
-  )
-  (wire (pts (xy 134.62 52.07) (xy 138.43 52.07))
+  (wire (pts (xy 104.14 120.65) (xy 104.14 125.73))
+    (stroke (width 0) (type default) (color 0 0 0 0))
+  )
+  (wire (pts (xy 104.14 125.73) (xy 107.95 125.73))
     (stroke (width 0) (type default) (color 0 0 0 0))
   )
@@
     (stroke (width 0) (type default) (color 0 0 0 0))
   )
-  (wire (pts (xy 121.92 110.49) (xy 121.92 113.03))
+  (wire (pts (xy 124.46 110.49) (xy 124.46 113.03))
     (stroke (width 0) (type default) (color 0 0 0 0))
   )
@@
     (stroke (width 0) (type default) (color 0 0 0 0))
   )
-  (wire (pts (xy 149.86 110.49) (xy 146.05 110.49))
-    (stroke (width 0) (type default) (color 0 0 0 0))
-  )
   (wire (pts (xy 85.09 59.69) (xy 83.82 59.69))
     (stroke (width 0) (type default) (color 0 0 0 0))
@@
     (stroke (width 0) (type default) (color 0 0 0 0))
   )
-  (wire (pts (xy 125.73 110.49) (xy 121.92 110.49))
+  (wire (pts (xy 128.27 110.49) (xy 124.46 110.49))
     (stroke (width 0) (type default) (color 0 0 0 0))
   )
@@
   )
   (wire (pts (xy 267.97 41.91) (xy 246.38 41.91))
+    (stroke (width 0) (type default) (color 0 0 0 0))
+  )
+  (wire (pts (xy 104.14 110.49) (xy 104.14 113.03))
     (stroke (width 0) (type default) (color 0 0 0 0))
   )
@@
     (stroke (width 0) (type default) (color 0 0 0 0))
   )
-  (wire (pts (xy 121.92 120.65) (xy 121.92 127))
+  (wire (pts (xy 124.46 120.65) (xy 124.46 127))
     (stroke (width 0) (type default) (color 0 0 0 0))
   )
@@
     (effects (font (size 1.27 1.27) (thickness 0.254) bold) (justify left bottom))
   )
-  (text "V-REG" (at 184.15 25.4 0)
+  (text "Power" (at 184.15 25.4 0)
     (effects (font (size 5 5)) (justify left bottom))
   )
@@
     (effects (font (size 5 5)) (justify left bottom))
   )
-  (global_label "EN" (shape input) (at 138.43 52.07 0) (fields_autoplaced)
-    (effects (font (size 1.27 1.27)) (justify left))
-    (property "Intersheet References" "${INTERSHEET_REFS}" (id 0) (at 143.3226 51.9906 0)
+  (global_label "EN" (shape input) (at 107.95 125.73 0) (fields_autoplaced)
+    (effects (font (size 1.27 1.27)) (justify left))
+    (property "Intersheet References" "${INTERSHEET_REFS}" (id 0) (at 112.8426 125.6506 0)
       (effects (font (size 1.27 1.27)) (justify left) hide)
     )
@@
     )
   )
-  (global_label "mGND" (shape input) (at 121.92 127 270) (fields_autoplaced)
-    (effects (font (size 1.27 1.27)) (justify right))
-    (property "Intersheet References" "${INTERSHEET_REFS}" (id 0) (at 121.9994 134.9769 90)
+  (global_label "mGND" (shape input) (at 124.46 127 270) (fields_autoplaced)
+    (effects (font (size 1.27 1.27)) (justify right))
+    (property "Intersheet References" "${INTERSHEET_REFS}" (id 0) (at 124.5394 134.9769 90)
       (effects (font (size 1.27 1.27)) (justify right) hide)
     )
@@
     )
   )
-  (global_label "io15" (shape input) (at 125.73 110.49 0) (fields_autoplaced)
-    (effects (font (size 1.27 1.27)) (justify left))
-    (property "Intersheet References" "${INTERSHEET_REFS}" (id 0) (at 132.316 110.4106 0)
+  (global_label "io15" (shape input) (at 128.27 110.49 0) (fields_autoplaced)
+    (effects (font (size 1.27 1.27)) (justify left))
+    (property "Intersheet References" "${INTERSHEET_REFS}" (id 0) (at 134.856 110.4106 0)
       (effects (font (size 1.27 1.27)) (justify left) hide)
     )
@@
     )
   )
-  (symbol (lib_id "Device:R") (at 134.62 43.18 0) (unit 1)
-    (in_bom yes) (on_board yes)
-    (property "Reference" "R2" (id 0) (at 136.398 42.0116 0)
-      (effects (font (size 1.27 1.27)) (justify left))
-    )
-    (property "Value" "10K" (id 1) (at 136.398 44.323 0)
-      (effects (font (size 1.27 1.27)) (justify left))
-    )
-    (property "Footprint" "Tinker:R_0603_1608Metric_Pad0.98x0.95mm_HandSolder" (id 2) (at 132.842 43.18 90)
-      (effects (font (size 1.27 1.27)) hide)
-    )
-    (property "Datasheet" "~" (id 3) (at 134.62 43.18 0)
+  (symbol (lib_id "Device:R") (at 104.14 116.84 0) (unit 1)
+    (in_bom yes) (on_board yes)
+    (property "Reference" "R2" (id 0) (at 105.918 115.6716 0)
+      (effects (font (size 1.27 1.27)) (justify left))
+    )
+    (property "Value" "10K" (id 1) (at 105.918 117.983 0)
+      (effects (font (size 1.27 1.27)) (justify left))
+    )
+    (property "Footprint" "Tinker:R_0603_1608Metric_Pad0.98x0.95mm_HandSolder" (id 2) (at 102.362 116.84 90)
+      (effects (font (size 1.27 1.27)) hide)
+    )
+    (property "Datasheet" "~" (id 3) (at 104.14 116.84 0)
       (effects (font (size 1.27 1.27)) hide)
     )
@@
     (pin "1")
   )
-  (symbol (lib_id "power:+3.3V") (at 149.86 110.49 0) (unit 1)
-    (in_bom yes) (on_board yes) (fields_autoplaced)
-    (property "Reference" "#PWR0121" (id 0) (at 149.86 114.3 0)
-      (effects (font (size 1.27 1.27)) hide)
-    )
-    (property "Value" "+3.3V" (id 1) (at 149.86 105.41 0))
-    (property "Footprint" "" (id 2) (at 149.86 110.49 0)
-      (effects (font (size 1.27 1.27)) hide)
-    )
-    (property "Datasheet" "" (id 3) (at 149.86 110.49 0)
+  (symbol (lib_id "power:+3.3V") (at 146.05 110.49 0) (unit 1)
+    (in_bom yes) (on_board yes) (fields_autoplaced)
+    (property "Reference" "#PWR0121" (id 0) (at 146.05 114.3 0)
+      (effects (font (size 1.27 1.27)) hide)
+    )
+    (property "Value" "+3.3V" (id 1) (at 146.05 105.41 0))
+    (property "Footprint" "" (id 2) (at 146.05 110.49 0)
+      (effects (font (size 1.27 1.27)) hide)
+    )
+    (property "Datasheet" "" (id 3) (at 146.05 110.49 0)
       (effects (font (size 1.27 1.27)) hide)
     )
@@
     (pin "2")
   )
-  (symbol (lib_id "Device:R") (at 121.92 116.84 0) (unit 1)
-    (in_bom yes) (on_board yes)
-    (property "Reference" "R7" (id 0) (at 123.698 115.6716 0)
-      (effects (font (size 1.27 1.27)) (justify left))
-    )
-    (property "Value" "10K" (id 1) (at 123.698 117.983 0)
-      (effects (font (size 1.27 1.27)) (justify left))
-    )
-    (property "Footprint" "Tinker:R_0603_1608Metric_Pad0.98x0.95mm_HandSolder" (id 2) (at 120.142 116.84 90)
-      (effects (font (size 1.27 1.27)) hide)
-    )
-    (property "Datasheet" "~" (id 3) (at 121.92 116.84 0)
+  (symbol (lib_id "Device:R") (at 124.46 116.84 0) (unit 1)
+    (in_bom yes) (on_board yes)
+    (property "Reference" "R7" (id 0) (at 126.238 115.6716 0)
+      (effects (font (size 1.27 1.27)) (justify left))
+    )
+    (property "Value" "10K" (id 1) (at 126.238 117.983 0)
+      (effects (font (size 1.27 1.27)) (justify left))
+    )
+    (property "Footprint" "Tinker:R_0603_1608Metric_Pad0.98x0.95mm_HandSolder" (id 2) (at 122.682 116.84 90)
+      (effects (font (size 1.27 1.27)) hide)
+    )
+    (property "Datasheet" "~" (id 3) (at 124.46 116.84 0)
       (effects (font (size 1.27 1.27)) hide)
     )
@@
     (pin "1")
   )
-  (symbol (lib_id "power:+3.3V") (at 134.62 39.37 0) (unit 1)
-    (in_bom yes) (on_board yes) (fields_autoplaced)
-    (property "Reference" "#PWR0106" (id 0) (at 134.62 43.18 0)
-      (effects (font (size 1.27 1.27)) hide)
-    )
-    (property "Value" "+3.3V" (id 1) (at 134.62 34.29 0))
-    (property "Footprint" "" (id 2) (at 134.62 39.37 0)
-      (effects (font (size 1.27 1.27)) hide)
-    )
-    (property "Datasheet" "" (id 3) (at 134.62 39.37 0)
-      (effects (font (size 1.27 1.27)) hide)
-    )
+  (symbol (lib_id "power:+3.3V") (at 104.14 110.49 0) (unit 1)
+    (in_bom yes) (on_board yes) (fields_autoplaced)
+    (property "Reference" "#PWR0106" (id 0) (at 104.14 114.3 0)
+      (effects (font (size 1.27 1.27)) hide)
+    )
+    (property "Value" "+3.3V" (id 1) (at 104.14 105.41 0))
+    (property "Footprint" "" (id 2) (at 104.14 110.49 0)
+      (effects (font (size 1.27 1.27)) hide)
+    )
+    (property "Datasheet" "" (id 3) (at 104.14 110.49 0)
+      (effects (font (size 1.27 1.27)) hide)
+    )
