File: Hardware/ESP-12/ESP12.kicad_pcb (KiCad board)
At the start: 2 copper layers, 71.3 x 61 mm, 36 parts, among them J1 USB_C_Receptacle_USB2.0, Q1 MMBT3904, Q2 MMBT3904, SW1 SW_Push, SW2 SW_DIP_x01, U1 CH340G, U2 AMS1117-3.3, Y1 12M

Commit message: Getting up to rev 1
Parts:
- removed the G*** at (163.1, 102.0)
- added R7: 10K, Tinker:R_0603_1608Metric_Pad0.98x0.95mm_HandSolder, F.Cu at (163.0, 89.0)
- added R8: 10K, Tinker:R_0603_1608Metric_Pad0.98x0.95mm_HandSolder, F.Cu at (165.0, 89.0)
- added REF**: DagNabbit, Rabbit:DagNabbit, F.Cu at (162.7, 100.0)
- moved R2 13.9 mm to (137.0, 89.0), turned to 90 degrees
- moved SW2 7.74 mm to (150.0, 97.5), turned to 180 degrees
- moved R1 6.37 mm to (143.0, 103.0)
- moved R5 4.60 mm to (157.0, 95.0), turned to 180 degrees
- moved R6 4.60 mm to (143.0, 95.0), turned to 0 degrees
- moved D1 3.18 mm to (157.0, 97.5), turned to 180 degrees
- moved D2 3.18 mm to (143.0, 97.5), turned to 0 degrees
- moved C1 1.51 mm to (136.0, 112.7)
- moved C2 1.51 mm to (136.0, 109.2)
- moved Y1 1.21 mm to (139.5, 111.0)
Connections:
- D2 pad 2: Vsw -> +3.3V
- R1 pad 1: Vsw -> +3.3V
- R2 pad 1: Vsw -> +3.3V
- R6 pad 2: GND -> mGND
- SW2 pad 1: Vsw -> GND
- SW2 pad 2: +3.3V -> mGND
- Um1 pad 10: unconnected-(Um1-Pad10) -> io15
- Um1 pad 11: io2 -> unconnected-(Um1-Pad11)
- Um1 pad 13: io4 -> unconnected-(Um1-Pad13)
- Um1 pad 4: io16 -> unconnected-(Um1-Pad4)
- Um1 pad 5: io14 -> unconnected-(Um1-Pad5)
- Um1 pad 6: io12 -> unconnected-(Um1-Pad6)
- Um1 pad 7: io13 -> unconnected-(Um1-Pad7)
- Um1 pad 8: Vsw -> +3.3V
- Um1 pad 9: GND -> mGND
Routing:
- net mGND: track 0.00 -> 29.5 mm
- net io0: track 23.2 -> 36.1 mm, vias 0 -> 1
- net EN: track 25.6 -> 15.1 mm
- net io15: track 0.00 -> 7.15 mm
- net Net-(C2-Pad1): track 6.41 -> 8.00 mm
- net unconnected-(Um1-Pad7): track 0.00 -> 1.55 mm
- net unconnected-(Um1-Pad6): track 0.00 -> 1.55 mm
- net unconnected-(Um1-Pad5): track 0.00 -> 1.55 mm
- net unconnected-(Um1-Pad4): track 0.00 -> 1.55 mm
- net unconnected-(Um1-Pad13): track 0.00 -> 1.55 mm
- net unconnected-(Um1-Pad11): track 0.00 -> 1.55 mm
- net unconnected-(Um1-Pad10): track 1.55 -> 0.00 mm
- net io4: track 1.55 -> 0.00 mm
- net io2: track 1.55 -> 0.00 mm
- net io16: track 1.55 -> 0.00 mm
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- removed copper zone on F.Cu, net Vsw
Other:
- board text added: "(v1.0.?)"
- board text added: "MOD POWER"
- board text removed: "(en)"
- board text removed: "(v0.5.2)"
- board text removed: "POWER"
