File: Hardware/ESP-12/ESP12.kicad_pcb (KiCad board)
At the start: 2 copper layers, 71.3 x 61 mm, 38 parts, among them J1 USB_C_Receptacle_USB2.0, Q1 MMBT3904, Q2 MMBT3904, SW1 SW_Push, SW2 SW_DIP_x01, U1 CH340G, U2 AMS1117-3.3, Y1 12M

Commit message: ...
Parts:
- removed G***: LOGO, Rabbit:rabbit
- added REF**: DagNabbit, Rabbit:DagNabbit, B.Cu at (149.6, 115.0)
Other:
- board text added: "You can put sticky stuff here. Or even, if you really feel like it, drill holes through this part. (I'd suggest verifying that the fasteners going through those holes have heads that don't stick up far enough to interfere with stuff...)"

Commit message: v1.0.0 gerbers submitted
Other:
- board text added: "(v1.0.0)"
- board text removed: "(v1.0.?)"
Changed lines of the file:
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@@
     (title "The Nerd Mage Module Programmer")
     (date "2023-07-13")
-    (rev "1.0.?")
+    (rev "1.0.0")
     (company "S. A. Miller")
     (comment 1 "ESP-12/07 Edition")
@@
     (effects (font (size 1.5 1.5) (thickness 0.3)) (justify mirror))
   )
-  (gr_text "(v1.0.?)" (at 150 101.997455) (layer "B.SilkS")
+  (gr_text "(v1.0.0)" (at 150 101.997455) (layer "B.SilkS")
     (effects (font (size 1 1) (thickness 0.15)) (justify mirror))
   )
