File: Hardware/Seeed Wio-RP2040/Wio-RP2040.kicad_pcb (KiCad board)
At the start: 2 copper layers, 71.3 x 66.5 mm, 36 parts, among them J1 USB_C_Receptacle_USB2.0, Q1 MMBT3904, Q2 MMBT3904, SW1 SW_Push, SW2 SW_DIP_x01, U1 CH340G, U2 AMS1117-3.3, Y1 12M

Commit message: werkin on da RP2040
Parts:
- removed C1, C2: 20p, Tinker:C_0603_1608Metric_Pad1.08x0.95mm_HandSolder
- removed C3: 10nf, Tinker:C_0603_1608Metric_Pad1.08x0.95mm_HandSolder
- removed C4: 100nf, Tinker:C_0603_1608Metric_Pad1.08x0.95mm_HandSolder
- removed C5: 22uf, Capacitor_Tantalum_SMD:CP_EIA-6032-28_Kemet-C_Pad2.25x2.35mm_HandSolder
- removed D1, D2: LED, LED_SMD:LED_0805_2012Metric_Pad1.15x1.40mm_HandSolder
- removed Q1, Q2: MMBT3904, Package_TO_SOT_SMD:SOT-23_Handsoldering
- removed R5, R6: 2K2, Tinker:R_0603_1608Metric_Pad0.98x0.95mm_HandSolder
- removed the REF** at (163.1, 94.0)
- removed the REF** at (199.3, 94.0)
- removed the REF** at (136.9, 94.0)
- removed the REF** at (173.1, 94.0)
- removed U1: CH340G, Package_SO:SOIC-16_3.9x9.9mm_P1.27mm
- removed U2: AMS1117-3.3, Package_TO_SOT_SMD:SOT-223-3_TabPin2
- removed Y1: 12M, Crystal:Crystal_SMD_5032-2Pin_5.0x3.2mm
- added SW3: SW_Push, Tinker:SW_Push_TS273014TP, F.Cu at (150.0, 110.0)
- moved SW2 21.1 mm to (162.7, 110.2)
- moved REF** 11.3 mm to (163.1, 73.2)
- moved REF** 11.3 mm to (136.9, 73.2)
- moved Um1 11.3 mm to (150.0, 83.3)
- moved R1 10.8 mm to (140.8, 107.1)
- moved REF** 10.2 mm to (173.1, 72.6)
- moved REF** 10.2 mm to (199.3, 72.6)
- moved R2 9.92 mm to (149.2, 107.1), turned to 180 degrees
- moved SW1 8.83 mm to (140.0, 110.0), turned to 0 degrees
Connections:
- R2 pad 2: EN -> mode
- SW2 pad 2: +3.3V -> Vcc
- Um1 pad 1: unconnected-(Um1-Pad1) -> GND
- Um1 pad 10: unconnected-(Um1-Pad10) -> mode
- Um1 pad 11: unconnected-(Um1-Pad11) -> RST
- Um1 pad 12: unconnected-(Um1-Pad12) -> GND
- Um1 pad 2: unconnected-(Um1-Pad2) -> Vsw
- Um1 pad 21: unconnected-(Um1-Pad21) -> GND
- Um1 pad 32: unconnected-(Um1-Pad32) -> GND
- Um1 pad 33: unconnected-(Um1-Pad33) -> GND
- Um1 pad 8: unconnected-(Um1-Pad8) -> UD-
- Um1 pad 9: unconnected-(Um1-Pad9) -> UD+
Routing:
- net mode: track 0.00 -> 22.7 mm
- net UD+: track 11.5 -> 33.2 mm, vias 2 -> 1
- net UD-: track 12.8 -> 34.0 mm, vias 2 -> 1
- net RTS: track 19.3 -> 0.00 mm, vias 2 -> 0
- net DTR: track 18.0 -> 0.00 mm, vias 2 -> 0
- net TxD: track 16.9 -> 0.00 mm, vias 1 -> 0
- net RxD: track 16.8 -> 0.00 mm, vias 1 -> 0
- net Net-(C1-Pad1): track 10.4 -> 0.00 mm
- net EN: track 7.66 -> 0.00 mm
- net RST: track 27.1 -> 19.5 mm, vias 1 -> 0
- net Vcc: track 14.7 -> 8.12 mm
- net Net-(C2-Pad1): track 6.41 -> 0.00 mm
- net +3.3V: track 2.24 -> 0.00 mm
- net Net-(D2-Pad1): track 2.03 -> 0.00 mm
- net Net-(D1-Pad1): track 2.03 -> 0.00 mm
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- removed copper zone on F.Cu, net +3.3V
- removed copper zone on F.Cu, net GND
Other:
- board size 71.3 x 66.5 mm -> 71.3 x 56.4 mm
- board text added: "(v0.0.666)"
- board text added: "MODE"
- board text added: "The Nerd Mage Module Programmer (sorta...)"
- board text removed: "(en)"
- board text removed: "(v0.5.2)"
- board text removed: "The Nerd Mage Module Programmer"
