File: Hardware/Pop-In RP2040/Pop-In RP2040.kicad_sch (KiCad schematic)
At the start: 25 parts, among them J1 USB_C_Receptacle_USB2.0, J2 Conn_01x06_Male, Q1 MMBT3904, Q2 MMBT3904, SW1 SW_Push, SW2 SW_DIP_x01, U1 CH340G, U2 AMS1117-3.3, Y1 12M

Commit message: ...
Other:
- note added: "This is not actually valid in ANY way. It is a placeholder."
- note removed: "100K"
- note removed: "10K"
Changed lines of the file:
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@@
     (rev "1.0.0")
     (company "S. A. Miller")
-    (comment 1 "ESP-12/07 Edition")
+    (comment 1 "Pop-In RP2040 Edition")
   )
   (junction (at 83.82 64.77) (diameter 0) (color 0 0 0 0)
@@
     (effects (font (size 5 5)) (justify left bottom))
   )
-  (text "100K" (at 215.9 48.26 0)
-    (effects (font (size 1.27 1.27)) (justify left bottom))
-  )
   (text "USB" (at 19.05 26.67 0)
     (effects (font (size 5 5)) (justify left bottom))
@@
     (effects (font (size 5 5)) (justify left bottom))
   )
-  (text "10K" (at 214.63 77.47 0)
-    (effects (font (size 1.27 1.27)) (justify left bottom))
+  (text "This is not\nactually valid\nin ANY way.\n\nIt is a placeholder."
+    (at 58.42 153.67 0)
+    (effects (font (size 12.7 12.7) (thickness 2.54) bold italic) (justify left bottom))
   )
   (text "RxD" (at 250.19 36.83 0)
